File: Archiv/CDTV-RAM-IDE-V0.5.sch (EAGLE design)
At the start: 56 parts, among them IC2 XC95288XL-TQ144, IC3 74HCT245PW, IC4 74HCT245PW, IC5 74HCT245PW, IC6 AS4C4M16S-6TCN, IC7 LD117AS33TR, IC8 AM29F010J-SOCKET

Commit message: Optimized the PCB and added a Jumper for AT-Bus/Oktapussy
Parts:
- C10, C11, C12, C19, C3, C4, C7, C8, C9: value (none) -> 100n
- F1: value 500mA -> 750mA
- IC10: value (none) -> 50MHz
- R1: value (none) -> FERRITE
- R4: value (none) -> 47
- RN1, RN10, RN2, RN3, RN4, RN5, RN6, RN7, RN8, RN9: value (none) -> 33
- RN11: value (none) -> 4.7k
Changed lines of the file:
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@@
 <part name="IC8" library="am29-memory" deviceset="AM29F010*" device="J-SOCKET" value="AM29F010J-SOCKET"/>
 <part name="IC9" library="micro-mc68000" deviceset="MC68000P" device="ROUND-PAD-BIG-HOLE"/>
-<part name="IC10" library="SMD-Crystal" deviceset="CSX-750FC" device="FC(5V)"/>
+<part name="IC10" library="SMD-Crystal" deviceset="CSX-750FC" device="FC(5V)" value="50MHz"/>
 <part name="C1" library="rcl" deviceset="C-EU" device="C0603K" value="100n"/>
 <part name="C2" library="rcl" deviceset="C-EU" device="C0805K" value="10u"/>
-<part name="C7" library="rcl" deviceset="C-EU" device="C0603K"/>
-<part name="C8" library="rcl" deviceset="C-EU" device="C0603K"/>
-<part name="C9" library="rcl" deviceset="C-EU" device="C0603K"/>
-<part name="C10" library="rcl" deviceset="C-EU" device="C0603K"/>
-<part name="C11" library="rcl" deviceset="C-EU" device="C0603K"/>
-<part name="C12" library="rcl" deviceset="C-EU" device="C0603K"/>
+<part name="C7" library="rcl" deviceset="C-EU" device="C0603K" value="100n"/>
+<part name="C8" library="rcl" deviceset="C-EU" device="C0603K" value="100n"/>
+<part name="C9" library="rcl" deviceset="C-EU" device="C0603K" value="100n"/>
+<part name="C10" library="rcl" deviceset="C-EU" device="C0603K" value="100n"/>
+<part name="C11" library="rcl" deviceset="C-EU" device="C0603K" value="100n"/>
+<part name="C12" library="rcl" deviceset="C-EU" device="C0603K" value="100n"/>
 <part name="C13" library="rcl" deviceset="C-EU" device="C0603K" value="100n"/>
 <part name="C14" library="rcl" deviceset="C-EU" device="C0603K" value="100n"/>
@@
 <part name="GND18" library="supply1" deviceset="GND" device=""/>
 <part name="GND19" library="supply1" deviceset="GND" device=""/>
-<part name="C19" library="rcl" deviceset="C-EU" device="C0603K"/>
-<part name="R1" library="rcl" deviceset="R-EU_" device="R0603"/>
+<part name="C19" library="rcl" deviceset="C-EU" device="C0603K" value="100n"/>
+<part name="R1" library="rcl" deviceset="R-EU_" device="R0603" value="FERRITE"/>
 <part name="+3V2" library="supply1" deviceset="+3V3" device=""/>
 <part name="+3V16" library="supply1" deviceset="+3V3" device=""/>
@@
 <part name="R2" library="rcl" deviceset="R-EU_" device="R0603" value="4.7k"/>
 <part name="R3" library="rcl" deviceset="R-EU_" device="R0603" value="4.7k"/>
-<part name="F1" library="rcl" deviceset="R-EU_" device="R2512" value="500mA"/>
+<part name="F1" library="rcl" deviceset="R-EU_" device="R2512" value="750mA"/>
 <part name="IC5" library="74xx-eu" deviceset="74*245" device="PW" technology="HCT" value="74HCT245PW"/>
 <part name="GND28" library="supply1" deviceset="GND" device=""/>
@@
 <part name="C23" library="rcl" deviceset="C-EU" device="C0805K" value="10u"/>
 <part name="GND21" library="supply1" deviceset="GND" device=""/>
-<part name="RN1" library="resistor-dil" deviceset="4R-N" device="CAY16"/>
-<part name="RN2" library="resistor-dil" deviceset="4R-N" device="CAY16"/>
-<part name="RN3" library="resistor-dil" deviceset="4R-N" device="CAY16"/>
-<part name="RN4" library="resistor-dil" deviceset="4R-N" device="CAY16"/>
-<part name="RN5" library="resistor-dil" deviceset="4R-N" device="CAY16"/>
-<part name="RN6" library="resistor-dil" deviceset="4R-N" device="CAY16"/>
-<part name="RN7" library="resistor-dil" deviceset="4R-N" device="CAY16"/>
-<part name="RN8" library="resistor-dil" deviceset="4R-N" device="CAY16"/>
+<part name="RN1" library="resistor-dil" deviceset="4R-N" device="CAY16" value="33"/>
+<part name="RN2" library="resistor-dil" deviceset="4R-N" device="CAY16" value="33"/>
+<part name="RN3" library="resistor-dil" deviceset="4R-N" device="CAY16" value="33"/>
+<part name="RN4" library="resistor-dil" deviceset="4R-N" device="CAY16" value="33"/>
+<part name="RN5" library="resistor-dil" deviceset="4R-N" device="CAY16" value="33"/>
+<part name="RN6" library="resistor-dil" deviceset="4R-N" device="CAY16" value="33"/>
+<part name="RN7" library="resistor-dil" deviceset="4R-N" device="CAY16" value="33"/>
+<part name="RN8" library="resistor-dil" deviceset="4R-N" device="CAY16" value="33"/>
 <part name="IC7" library="v-reg" deviceset="LD117A?*" device="S" technology="33TR"/>
-<part name="R4" library="rcl" deviceset="R-EU_" device="R0603"/>
+<part name="R4" library="rcl" deviceset="R-EU_" device="R0603" value="47"/>
 <part name="AUTOBOOT_OFF" library="jumper" deviceset="JP1E" device=""/>
 <part name="R5" library="rcl" deviceset="R-EU_" device="R0603" value="4.7k"/>
-<part name="RN9" library="resistor-dil" deviceset="4R-N" device="CAY16"/>
-<part name="RN10" library="resistor-dil" deviceset="4R-N" device="CAY16"/>
+<part name="RN9" library="resistor-dil" deviceset="4R-N" device="CAY16" value="33"/>
+<part name="RN10" library="resistor-dil" deviceset="4R-N" device="CAY16" value="33"/>
 <part name="MEM_OFF" library="jumper" deviceset="JP1E" device=""/>
 <part name="ACT" library="jumper" deviceset="JP1E" device=""/>
@@
 <part name="R6" library="rcl" deviceset="R-EU_" device="R0603" value="4.7k"/>
 <part name="R7" library="rcl" deviceset="R-EU_" device="R0603" value="330"/>
-<part name="C3" library="rcl" deviceset="C-EU" device="C0603K"/>
+<part name="C3" library="rcl" deviceset="C-EU" device="C0603K" value="100n"/>
 <part name="GND22" library="supply1" deviceset="GND" device=""/>
 <part name="+3V17" library="supply1" deviceset="+3V3" device=""/>
-<part name="C4" library="rcl" deviceset="C-EU" device="C0603K"/>
+<part name="C4" library="rcl" deviceset="C-EU" device="C0603K" value="100n"/>
 <part name="GND24" library="supply1" deviceset="GND" device=""/>
 <part name="+3V18" library="supply1" deviceset="+3V3" device=""/>
 <part name="R8" library="rcl" deviceset="R-EU_" device="R0603" value="4.7k"/>
-<part name="RN11" library="resistor-dil" deviceset="4R-N" device="CAY16"/>
+<part name="RN11" library="resistor-dil" deviceset="4R-N" device="CAY16" value="4.7k"/>
 </parts>
 <sheets>
